File: CCFL2LED.kicad_pcb (KiCad board)
At the start: 2 copper layers, 55.1 x 85.1 mm, 68 parts, among them J2 USB_C_Receptacle_USB2.0_16P, J3 Jack-DC, J4 OUTPUT, J7 Conn_01x02_Pin, Q1 S8050, SW1 SW_SPDT, U1 PT4115, U2 PT4115, U3 AP62201WU-7, U7 LM2596 Modul, U8 AMS1117-3.3, U9 CH224K

Commit message: Trace update
- Update pictures
- Update kicad_pcb
- Update fabrication files
Parts:
- moved Q1 0.70 mm to (72.6, 106.1), turned to -90 degrees
- moved F2 0.24 mm to (82.8, 49.6)
Routing:
- net GND: track 0.00 -> 26.5 mm
- net +12V: track 195.4 -> 189.3 mm
- net /Vdd: track 17.6 -> 20.8 mm
- net /DimPin: track 8.43 -> 6.05 mm
- net /CC2: track 7.61 -> 8.78 mm, vias 0 -> 2
- net /emitor: track 2.05 -> 3.16 mm
- net /Base: track 48.4 -> 47.3 mm
- net /D+: track 18.2 -> 17.3 mm
- net /Vbus: track 37.4 -> 36.5 mm
- net /CC1: track 5.15 -> 5.45 mm, vias 2 -> 0
